File: ThumbsUp.kicad_pcb (KiCad board)
At the start: 2 copper layers, 342 x 336.1 mm, 139 parts, among them J1 Conn_01x04_Male, J10 Raiser_Male, J11 Raiser_Female, J12 Raiser_Male, J13 Raiser_Female, J14 Raiser_Male, J15 Raiser_Female, J16 Raiser_Male, J17 Raiser_Female, J18 Raiser_Male, J19 52559-1233, J2 Conn_01x04_Male, J20 Conn_01x04_Female, J21 Conn_01x04_Female, J22 Conn_01x04_Female, J23 Conn_01x04_Female, J24 Conn_01x04_Male, J25 Conn_01x04_Male, J26 Conn_01x04_Male, J27 Conn_01x04_Male, J28 Conn_01x04_Female, J29 Conn_01x04_Female, J3 Conn_01x04_Female, J30 Conn_01x04_Female, J31 Conn_01x04_Female, J32 Battery, J33 Conn_01x04_Female, J34 Conn_01x04_Female, J35 Raiser_Female, J36 Raiser_Female, J37 Raiser_Female, J38 52559-1233, J4 Conn_01x04_Male, J5 Conn_01x04_Female, J6 Conn_01x04_Male, J7 Conn_01x04_Male, J8 Conn_01x04_Male, J9 Raiser_Female, SW1 SW_Push, SW2 SW_DIP_x01, U1 ProMicro

Commit message: v9 Redrew the lower PCB, added the silkscreens.
Parts:
- added G***: LOGO, Silkscreens:Crowfeet75, F.Cu at (149.3, 52.1)
- added G***: LOGO, Silkscreens:Crowfeet75, F.Cu at (148.9, -74.7)
- added G***: LOGO, Silkscreens:Crowfeet75, F.Cu at (146.1, 183.8)
- added G***: LOGO, Silkscreens:Crowfeet75, F.Cu at (144.4, 321.7)
- added G***: LOGO, Silkscreens:Crowfeet75, B.Cu at (145.5, 322.3)
- moved J33 197.1 mm to (85.0, -34.2)
- moved J34 197.1 mm to (214.7, -34.3)
- moved J35 197.1 mm to (118.5, -22.9)
- moved J36 197.1 mm to (149.7, -72.7)
- moved J37 197.1 mm to (180.9, -23.1)
- moved J38 197.1 mm to (173.2, -28.2)
- moved MX45 197.1 mm to (124.7, -16.5)
- moved MX46 197.1 mm to (174.7, -16.7)
- moved MX47 197.1 mm to (108.7, -28.5)
- moved MX48 197.1 mm to (94.0, -39.6)
- moved MX49 197.1 mm to (205.7, -39.7)
- moved MX50 197.1 mm to (190.9, -28.5)
Connections:
- J12 pad 1: (no net) -> GND_L1
- J12 pad 2: (no net) -> GND_L1
- J12 pad 3: (no net) -> GND_L1
- J12 pad 4: (no net) -> GND_L1
- J16 pad 1: (no net) -> GND_L1
- J16 pad 2: (no net) -> GND_L1
- J16 pad 3: (no net) -> GND_L1
- J16 pad 4: (no net) -> GND_L1
Routing:
- net Net-(J1-Pad3): track 107.5 -> 76.0 mm, vias 1 -> 0
- net Net-(J1-Pad4): track 130.2 -> 99.8 mm
- net Net-(J28-Pad1): track 115.7 -> 85.4 mm, vias 2 -> 1
- net Net-(J1-Pad2): track 96.8 -> 74.0 mm, vias 0 -> 1
- net Net-(J28-Pad4): track 126.8 -> 104.9 mm, vias 0 -> 2
- net Net-(J28-Pad2): track 95.0 -> 73.3 mm
- net Net-(J28-Pad3): track 102.7 -> 82.0 mm, vias 2 -> 0
- net Net-(J1-Pad1): track 107.9 -> 88.5 mm, vias 0 -> 1
- net Net-(J30-Pad1): track 112.9 -> 98.9 mm, vias 0 -> 1
- net Net-(J29-Pad4): track 27.4 -> 39.1 mm, vias 0 -> 1
- net Net-(J2-Pad2): track 84.9 -> 73.8 mm, vias 0 -> 1
- net Net-(J2-Pad3): track 61.7 -> 50.8 mm, vias 0 -> 1
- net Net-(J30-Pad4): track 25.9 -> 36.3 mm, vias 0 -> 1
- net Net-(J8-Pad3): track 53.2 -> 62.2 mm, vias 0 -> 1
- net Net-(J2-Pad1): track 94.9 -> 103.4 mm, vias 0 -> 1
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- added copper zone on B.Cu, net GND_L1
Other:
- board size 342 x 336.1 mm -> 251.1 x 457.9 mm
