File: ThumbsUp.kicad_pcb (KiCad board)
At the start: 2 copper layers, 251.1 x 457.9 mm, 144 parts, among them J1 Conn_01x04_Male, J10 Raiser_Male, J11 Raiser_Female, J12 Raiser_Male, J13 Raiser_Female, J14 Raiser_Male, J15 Raiser_Female, J16 Raiser_Male, J17 Raiser_Female, J18 Raiser_Male, J19 52559-1233, J2 Conn_01x04_Male, J20 Conn_01x04_Female, J21 Conn_01x04_Female, J22 Conn_01x04_Female, J23 Conn_01x04_Female, J24 Conn_01x04_Male, J25 Conn_01x04_Male, J26 Conn_01x04_Male, J27 Conn_01x04_Male, J28 Conn_01x04_Female, J29 Conn_01x04_Female, J3 Conn_01x04_Female, J30 Conn_01x04_Female, J31 Conn_01x04_Female, J32 Battery, J33 Conn_01x04_Female, J34 Conn_01x04_Female, J35 Raiser_Female, J36 Raiser_Female, J37 Raiser_Female, J38 52559-1233, J4 Conn_01x04_Male, J5 Conn_01x04_Female, J6 Conn_01x04_Male, J7 Conn_01x04_Male, J8 Conn_01x04_Male, J9 Raiser_Female, SW1 SW_Push, SW2 SW_DIP_x01, U1 ProMicro

Commit message: v9 Redrew the lower PCB, added the silkscreens.
Parts:
- moved G*** 85.1 mm to (149.3, 236.7)
- moved J12 85.1 mm to (195.0, 278.4)
- moved J16 85.1 mm to (99.0, 273.9)
- moved J30 85.1 mm to (183.8, 216.4)
- moved J31 85.1 mm to (190.3, 232.9)
- moved MX7 85.1 mm to (83.4, 188.8)
- moved D1 85.1 mm to (147.4, 133.5)
- moved D10 85.1 mm to (116.0, 123.0)
- moved D11 85.1 mm to (118.4, 123.0)
- moved D12 85.1 mm to (120.8, 123.0)
- moved D13 85.1 mm to (108.9, 123.0)
- moved D14 85.1 mm to (106.5, 123.0)
- moved D15 85.1 mm to (147.4, 135.9)
- moved D16 85.1 mm to (139.8, 135.9)
- moved D17 85.1 mm to (111.3, 123.0)
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